Commit message: kk

File: assets/ur5/doosan_origin.urdf (robot description, URDF)
Before this commit: robot Doosan_loz, 13 links, 12 joints
Links:
- removed link base
- removed link ee_link
- removed link tool0
- removed link tool_tip
- removed link world
Joints:
- removed joint base_link-base_fixed_joint
- removed joint ee_fixed_joint
- removed joint tool0_fixed_joint-tool_tip
- removed joint world_joint
- removed joint wrist_3_link-tool0_fixed_joint
- joint joint3: limit lower=-2.617993878 upper=2.617993878 effort=150.0 velocity=3.141592654 -> lower=-6.28318530718 upper=6.28318530718 effort=150.0 velocity=3.141592654
- joint rotated_base-base_fixed_joint: origin xyz=0.0 0.0 0.0 rpy=0.0 0.0 0.0 -> xyz=0.0 0.0 0.0 rpy=0.0 0.0 0
