Commit message: update_line

File: assets/objects/rod.urdf (robot description, URDF)
Before this commit: robot custom, 1 links, 0 joints
Links:
- added link sphere_1, mass 0; collision sphere radius=0.01; visual sphere radius=0.01
- added link sphere_2, mass 0; collision sphere radius=0.01; visual sphere radius=0.01
- link base_link: mass 0.05 -> 0.1
Joints:
- added joint joint_1: type fixed, parent base_link, child sphere_1, origin xyz=0 0.08 0
- added joint joint_2: type fixed, parent base_link, child sphere_2, origin xyz=-0 -0.08 0

File: assets/obstacles/block.urdf (robot description, URDF)
Before this commit: robot simple_cuboid, 1 links, 0 joints
Links:
- link base_link: geometry collision box size=0.1 0.1 0.1; visual box size=0.1 0.1 0.1

Commit message: add force

File: assets/objects/rod.urdf (robot description, URDF)
Before this commit: robot custom, 3 links, 2 joints
Links:
- link sphere_1: geometry collision sphere radius=0.001; visual sphere radius=0.001
- link sphere_2: geometry collision sphere radius=0.001; visual sphere radius=0.001
