Commit message: fix base-cabin-bin

File: assets/obstacles/block.urdf (robot description, URDF)
Before this commit: robot simple_cuboid, 1 links, 0 joints
Links:
- link base_link: geometry collision box size=0.2 0.2 0.2; visual box size=0.1 0.1 0.1

File: assets/ur5/base_doosan.urdf (robot description, URDF)
Before this commit: robot m0609, 2 links, 1 joints
Links:
- removed link base
Joints:
- removed joint fixed

Commit message: two_tree

File: assets/obstacles/block.urdf (robot description, URDF)
Before this commit: robot simple_cuboid, 1 links, 0 joints
Links:
- link base_link: geometry collision box size=0.3 0.3 0.3; visual box size=0.3 0.3 0.3
